File: PCB/PyBoardTester.kicad_sch (KiCad schematic)
At the start: 47 parts, among them J1 6pin_hd, J4 3pin_hd, J5 USB4105-GF-A, SW1 SW_SPST, U4 ATXMEGA32A4U-MH, U7 FT232RNL, U8 LP5907MFX-3.3

Commit message: modificado power-jumper
- passou a ser solder-jumper
- default: ligado a USB-Power
Parts:
- J4: footprint Connector_PinHeader_2.54mm:PinHeader_1x03_P2.54mm_Vertical -> Jumper:SolderJumper-3_P1.3mm_Bridged12_RoundedPad1.0x1.5mm
Changed lines of the file:
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@@
 			)
 		)
-		(property "Footprint" "Connector_PinHeader_2.54mm:PinHeader_1x03_P2.54mm_Vertical"
+		(property "Footprint" "Jumper:SolderJumper-3_P1.3mm_Bridged12_RoundedPad1.0x1.5mm"
 			(at 63.5 193.04 0)
 			(effects

Commit message: após revisão do Filipe
- adicionados LEDs PASS & FAIL para sinalizar fim teste
- modificadasa Designators de LEDs para estar coerente na BOM
- unidos pares de IOs do pyBoard q faltavam
- reimensionado divisor resistivo para ADC-In
Parts:
- added D10: Green LED, LED_SMD:LED_0603_1608Metric, symbol Device:LED
- added D11: Red LED, LED_SMD:LED_0603_1608Metric, symbol Device:LED
- added R35: 330R, Resistor_SMD:R_0402_1005Metric, symbol Device:R_US
- added R36: 560, Resistor_SMD:R_0402_1005Metric, symbol Device:R_US
- C15, C26, C27, C29, C5, C6, C7, C8: footprint Capacitor_SMD:C_0402_1005Metric_Pad0.74x0.62mm_HandSolder -> Capacitor_SMD:C_0402_1005Metric; MPN C1005X7R1E104K050BB -> CGA2B3X7R1H104K050BB; OEPSPN OEPS010050 -> OEPS010016
- D1: value STATE-LED -> Green LED; MPN 5990010007F -> LTST-C191KGKT; OEPSPN OEPS030044 -> OEPS030005
- D2: value A-PWR -> Green LED; MPN 5990010007F -> LTST-C191KGKT; OEPSPN OEPS030044 -> OEPS030005
- D3: value B-PWR -> Green LED; MPN 5990010007F -> LTST-C191KGKT; OEPSPN OEPS030044 -> OEPS030005
- D4: value C-PWR -> Green LED; MPN 5990010007F -> LTST-C191KGKT; OEPSPN OEPS030044 -> OEPS030005
- D5, D6, D7, D8, D9: value D-PWR -> Green LED; MPN 5990010007F -> LTST-C191KGKT; OEPSPN OEPS030044 -> OEPS030005
- R21, R22, R23, R24, R25, R26, R28, R33, R34: value 560R -> 330R; MPN CRCW0402560RFKED -> CRCW0402330RFKEDHP; OEPSPN OEPS020193 -> OEPS020191
- R29, R30: value 5.1k -> 5k1
- R38: MPN CRCW040210K0FKED -> CPF0402B10KE1; OEPSPN OEPS020030 -> OEPS020043
Connections:
- net GND: now also D10.1 (K), D11.1 (K)
- net OK_LED: now reaches U4.10 (PC0/OC0A/SDA)
- net OK_LED: now also R35.2
- net NOK_LED: now reaches U4.11 (PC1/OC0B/XCK0/SCL)
- net NOK_LED: now also R36.2
- new net: D10.2 (A), R35.1
- new net: D11.2 (A), R36.1
- no-connect marks 23 -> 21
