File: PCB/OE PyBoard tester.kicad_pcb (KiCad board)
At the start: 4 copper layers, 113.5 x 114.7 mm, 117 parts, among them J1 6pin_hd, J2 Conn_01x08, J3 Conn_01x08, J4 3pin_hd, J5 USB4105-GF-A, SW1 SW_SPST, U1 THS4281, U3 THS4281, U4 ATXMEGA32A4U-MH, U5 THS4281, U6 THS4281, U7 FT232RNL, U8 LP5907MFX-3.3

Commit message: modificado nome projecto - OE PyBoard tester
OE PyBoard tester
- feita nova anotação para componentes ficarem com Referências sem jumps
- novo nome às Symbol & Footprint Libraries
- optimizadas link de componentes & footprints às novas Libraries
- retirado campo 'values' de Fab. Layer
- gerados novos ficheiros de produção: Gerbers & Drills & P&P & .d356 & BOM
Parts:
- J1: renamed from J5; footprint Connector_USB:USB_C_Receptacle_GCT_USB4105-xx-A_16P_TopMnt_Horizontal -> PyBoardTester FootprintLib:USB_C_Receptacle_GCT_USB4105-xx-A_16P_TopMnt_Horizontal
- X1: renamed from OSC1; footprint _footprintLib:OSC -> PyBoardTester FootprintLib:OSC
- renumbered C5 to C1, C15 to C10, C18 to C11, C28 to C12, C32 to C13, C34 to C14, C14 to C15, C13 to C16, C9 to C17, C10 to C18, C17 to C19, C8 to C2, C16 to C20, C11 to C21, C12 to C22, C1 to C23, C2 to C24, C3 to C25, C4 to C26, C7 to C3, C6 to C4, C30 to C5, C31 to C6, C29 to C7, C27 to C8, C26 to C9, J1 to J2, J4 to J3, J2 to J4, J3 to J5, R29 to R1, R24 to R10, R25 to R11, R26 to R12, R28 to R13, R33 to R14, R34 to R15, R35 to R16, R36 to R17, R30 to R2, R13 to R22, R1 to R23, R15 to R24, R14 to R25, R2 to R26, R3 to R27, R16 to R28, R4 to R29, R31 to R3, R17 to R30, R5 to R31, R19 to R32, R18 to R33, R6 to R34, R7 to R35, R20 to R36, R10 to R37, R32 to R4, R27 to R5, R38 to R6, R21 to R7, R22 to R8, R23 to R9, U4 to U1, U7 to U2, U8 to U3, U1 to U6, U6 to U7, U3 to U8
Routing:
- net GND: track 111.5 -> 110.5 mm
- net +3V3#2: track 46.5 -> 45.6 mm
Other:
- board text added: "C7"
- board text added: "R29"
