File: PCB/OE PyBoard tester.kicad_pcb (KiCad board)
At the start: 4 copper layers, 113.5 x 114.7 mm, 117 parts, among them J1 USB4105-GF-A, J2 6pin_hd, J3 3pin_hd, J4 Conn_01x08, J5 Conn_01x08, SW1 SW_SPST, U1 ATXMEGA32A4U-MH, U2 FT232RNL, U3 LP5907MFX-3.3, U5 THS4281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

Commit message: synchronizing with main branch
Parts:
- added NOK1: SW_SPST, Button_Switch_SMD:SW_SPST_TL3305B, F.Cu at (188.8, 69.2)
- added OK1: SW_SPST, Button_Switch_SMD:SW_SPST_TL3305B, F.Cu at (178.9, 69.2)
- R1, R2, R28, R29, R36, R37: value 5k1 -> 5k1 0.1%
- R22, R23, R24, R25, R26, R27, R30, R31, R32, R33, R34, R35, R6: value 10k -> 10k 0.1%
- moved R16 32.6 mm to (179.7, 112.5), turned to -90 degrees
- moved R17 29.3 mm to (181.8, 112.5), turned to -90 degrees
- moved D10 19.9 mm to (179.3, 98.3)
- moved D11 15.2 mm to (189.2, 98.3)
- moved R12 14.4 mm to (182.9, 78.4)
- moved R14 14.4 mm to (182.9, 84.8)
- moved D6 14.4 mm to (187.1, 78.4)
- moved D7 14.4 mm to (187.1, 81.6)
- moved D8 14.4 mm to (187.1, 84.9)
- moved D9 14.4 mm to (187.1, 88.1)
- moved R13 14.4 mm to (182.9, 81.6)
- moved R15 14.4 mm to (182.9, 88.1)
Connections:
- U1 pad 12: unconnected-(U1-PC2/OC0C/RXD0-Pad12) -> Net-(U1-PC2/OC0C/RXD0)
- U1 pad 13: unconnected-(U1-PC3/OC0D/TXD0-Pad13) -> Net-(U1-PC3/OC0D/TXD0)
Routing:
- net Net-(U1-PC2/OC0C/RXD0): track 0.00 -> 158.2 mm, vias 0 -> 3
- net Net-(U1-PC3/OC0D/TXD0): track 0.00 -> 148.6 mm, vias 0 -> 3
- net /OK_LED: track 109.8 -> 76.3 mm
- net /NOK_LED: track 106.0 -> 75.3 mm
- net Net-(D11-A): track 2.86 -> 20.0 mm
- net /SUPPLY_LED: track 115.3 -> 100.9 mm
- net /RST#1_LED: track 125.8 -> 111.4 mm
- net /RST#2_LED: track 121.0 -> 106.6 mm
- net /IOs_LED: track 109.9 -> 95.5 mm
- net Net-(D10-A): track 2.89 -> 14.1 mm
- net GND: track 110.5 -> 106.4 mm, vias 244 -> 254
- added copper zone on F.Cu, net GND
Other:
- board text added: "DUT 4 LEDs sequence OK?"
- board text added: "FINAL RESULT"
- board text added: "PyBoard Tester rev.A"
- board text added: "START"
- board text removed: "PyBoardTester rev.A"
